File: stm32_mather.sch (EAGLE design)
At the start: 56 parts

Commit message: デバッガを組み込む方式に変更 3.3vのリニアレギュレータを単純化
Parts:
- removed C15: 0.1u, rcl:C-EUC1608
- removed C16: (no value), rcl:C-EUC1608
- removed C5: 4.7u, rcl:C-EUC2012
- removed C6: 470p, rcl:C-EUC1608
- removed C7: 10u, rcl:C-EUC2012
- removed IC1: (no value), user_ic:CH340E
- removed LED1: (no value), user_leds:1608LED
- removed R1: 33k, user_rcl:R_REG
- removed R10, R14, R15, R9: 10k, user_rcl:R_REG
- removed R2: 20k, user_rcl:R_REG
- removed R6, R7: 5.1k, user_rcl:R_REG
- removed R8: 1k, user_rcl:R_REG
- removed U$14: FDC6305, user_tr_fet_igbt:FDC6305
- removed U$22: BOX14P, user_conector:BOX14P
- removed USB1: (no value), user_conector:USB_TYPE_C
- C3: value 0.22u -> 1u; device rcl:C-EUC2012 -> rcl:C-EUC1608
- C4: value 0.1u -> 2.2u
- U$10: value NJM11100 -> NJM2845; device user_ic:NJM11100 -> user_ic:NJM2845
- U$11: value 2SC5964 -> STLINKV3MODS; device user_tr_fet_igbt:2SC5964 -> user_ic:STLINKV3MODS
Connections:
- removed net N$1: C6.2, R1.1, R2.2, U$10.PIN5_VADJ
- removed net N$17: IC1.1_UD+, USB1.A6_DP1, USB1.B6_DP2
- removed net N$18: IC1.2_UD-, USB1.A7_DN1, USB1.B7_DN2
- removed net N$2: C4.1, U$10.PIN3_NOIS?
- removed net N$20: R7.2, USB1.A5_CC1
- removed net N$21: R6.2, USB1.B5_CC2
- removed net N$22: IC1.6_TNOU, R8.1
- removed net N$23: LED1.A, R8.2
- removed net N$24: C15.1, IC1.10_V3
- removed net N$25: IC1.4_RTS#, IC1.5_CTS#
- removed net N$26: IC1.8_TXD, R10.2, U$14.PIN2_S2
- removed net N$28: IC1.9_RXD, R9.1, U$14.PIN5_S1
- removed net N$3: C5.1, C6.1, U$10.PIN4_VOUT, U$11.B
- removed net USART1_RX: MCU1.59_PB7>, R14.1, U$14.PIN4_D2
- removed net USART1_TX: MCU1.58, R15.1, U$14.PIN6_D1
- net GND: now also U$10.GND, U$11.24_GND, U$11.26_GND, U$11.27_GND, U$11.29_GND, U$11.5_GNDDETECT, U$11.8_GND; no longer C15.2, C16.2, C5.2, C7.2, IC1.3_GND, LED1.K, R2.1, R6.1, R7.1, U$10.PIN2_GND, U$22.P$11, U$22.P$5, U$22.P$7, USB1.A12_B1_GND, USB1.A1_B12_GND
- net JTCK: now also U$11.13_T_JCLK/T_SWCLK; no longer U$22.P$6
- net JTDI: now also U$11.28_T_JTDI/NC; no longer U$22.P$10
- net JTDO: now also U$11.6_T_JTDO/T_SWO; no longer U$22.P$8
- net JTMS: now also U$11.4_T_JTMS/T_SWDIO; no longer U$22.P$4
- net NRST: now also U$11.31_T_NRST; no longer U$22.P$12
- net RX: now also U$11.15_T_VCP_RX; no longer U$22.P$13
- net TX: now also U$11.12_T_VCP_TX; no longer U$22.P$14
- net V3.3: now also C4.1, U$10.VOUT, U$11.30_T_VCC; no longer C7.1, R1.2, R14.2, R15.2, U$11.E, U$22.P$3
- net V5: now also U$10.VIN; no longer C16.1, IC1.7_VCC, R10.1, R9.2, U$10.PIN1_CON, U$10.PIN6_VIN, U$11.C, U$14.PIN1_G1, U$14.PIN3_G2, USB1.A4_B9_VBUS, USB1.A9_B4_VBUS
Other:
- note removed: "片方向の通信だから分圧か抵抗と高速ダイオードでレベル変換するんでいい気がする"
- moved on the sheet: C13, C14, C3, C4, JP1, LED2, R13, R16, R4, R5, R_I1, U$1

Commit message: 基板図の設計完了
Parts:
- R_I1: value (none) -> 1k
Connections:
- removed net N$13: C12.2, MCU1.18_VSS
- removed net N$14: C12.1, MCU1.19_VDD
- removed net N$15: C11.1, MCU1.47_VSS
- removed net N$16: C11.2, MCU1.48_VDD
- removed net N$30: C10.2, C2.2, MCU1.13_VDDA, U$12.PIN1
- removed net N$5: C9.1, MCU1.32_VDD
- removed net N$7: C2.1, MCU1.12_VSSA
- removed net N$8: C8.1, MCU1.64_VDD
- removed net N$9: C8.2, MCU1.63_VSS
- net GND: now also C10.2, C11.1, C12.2, C2.1, C8.2, MCU1.12_VSSA, MCU1.18_VSS, MCU1.47_VSS, MCU1.63_VSS, U$1.23_GND, U$1.4_GND, U$12.PIN1, U$15.B_K, U$15.G_K, U$15.R_K; no longer U$15.B_A, U$15.G_A, U$15.R_A
- net N$10: now also U$15.R_A; no longer U$15.R_K
- net N$29: now also U$15.G_A; no longer U$15.G_K
- net N$31: now also U$15.B_A; no longer U$15.B_K
- net V3.3: now also C11.2, C12.1, C2.2, C8.1, C9.1, MCU1.13_VDDA, MCU1.19_VDD, MCU1.32_VDD, MCU1.48_VDD, MCU1.64_VDD
